Commit message: Ros Package for Introduction to Vision and Robotics course -- first commit, lab 1

File: urdf/robot.urdf (robot description, URDF)
Before this commit: robot myrobot, 6 links, 5 joints
Links:
- added link base, mass 100; collision cylinder length=1 radius=1; visual cylinder length=1 radius=1
- added link dummy
- added link sphere_base, mass 0.00001; collision sphere radius=0.7; visual sphere radius=0.7
- link link0: mass 10 -> 1
- link link1: mass 0.1 -> 0.3
Joints:
- added joint base_to_link0: type revolute, parent base, child link0, origin xyz=0 0 1 rpy=0 0 0, axis 1 0 0, limit lower=-${pi/2} upper=${pi/2} effort=1000.0 velocity=5
- added joint dummy_joint: type fixed, parent dummy, child base
- added joint sphere_base_to_base: type fixed, parent base, child sphere_base, origin xyz=0 0 1 rpy=0 0 0
- joint link0_to_link1: limit lower=-${pi/2} upper=${pi/2} effort=1000.0 velocity=0.5 -> lower=-${pi/2} upper=${pi/2} effort=1000.0 velocity=5
- joint link1_to_link2: limit lower=-${pi/2} upper=${pi/2} effort=1000.0 velocity=0.5 -> lower=-${pi/2} upper=${pi/2} effort=1000.0 velocity=5

Commit message: Update robot.urdf

File: urdf/robot.urdf (robot description, URDF)
Before this commit: robot myrobot, 9 links, 8 joints
Links:
- link base: geometry collision cylinder length=1 radius=0.8; visual cylinder length=1 radius=0.8
- link link0: geometry collision cylinder length=3 radius=0.35; visual cylinder length=3 radius=0.35
- link link1: geometry collision cylinder length=3 radius=0.2; visual cylinder length=3 radius=0.2
- link sphere2: geometry collision sphere radius=0.3; visual sphere radius=0.3
Joints:
- removed joint sphere0_to_link0
- removed joint sphere1_to_link1
- removed joint sphere_base_to_base
- added joint sphere0_to_link1: type fixed, parent link1, child sphere0, origin xyz=0 0 0 rpy=0 0 0
- added joint sphere1_to_link2: type fixed, parent link2, child sphere1, origin xyz=0 0 0 rpy=0 0 0
- added joint sphere_base_to_link0: type fixed, parent link0, child sphere_base, origin xyz=0 0 0 rpy=0 0 0

Commit message: Update robot.urdf

File: urdf/robot.urdf (robot description, URDF)
Before this commit: robot myrobot, 9 links, 8 joints
Links:
- link base: mass 100 -> 1000
